File: blocks/composite/regulated_cascoded_cmirror/design_proposal/circuit_dia.kicad_sch (KiCad schematic)
At the start: 25 parts, among them Q1 PMOS, Q10 PMOS, Q11 NMOS, Q12 PMOS, Q13 NMOS, Q2 PMOS, Q20 NMOS, Q21 NMOS, Q22 NMOS, Q23 NMOS, Q24 NMOS, Q25 NMOS, Q26 NMOS, Q27 NMOS, Q28 NMOS, Q29 NMOS, Q3 PMOS, Q30 NMOS, Q31 NMOS, Q4 NMOS, Q5 NMOS, Q6 NMOS, Q7 PMOS, Q8 PMOS, Q9 NMOS

Commit message: updated scheatic
Other:
- note added: "OTA1"
- note added: "OTA2"
Changed lines of the file:
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@@
 		)
 	)
-	(text "Power"
+	(text "OTA2"
 		(exclude_from_sim no)
 		(at 185.166 27.178 0)
@@
 		)
 	)
-	(text "Power"
+	(text "OTA1"
 		(exclude_from_sim no)
 		(at 74.422 26.416 0)
